File: EEG_cap_final.brd (EAGLE design)
At the start: 132 x 105 mm, 150 parts, among them J1 2908-05WB-MG, J10 POWER_JACKPTH_LOCK, J11 POWER_JACKPTH_LOCK, J12 POWER_JACKPTH_LOCK, J13 POWER_JACKPTH_LOCK, J14 POWER_JACKPTH_LOCK, J15 POWER_JACKPTH_LOCK, J16 POWER_JACKPTH_LOCK, J17 POWER_JACKPTH_LOCK, J18 POWER_JACKPTH_LOCK, J19 POWER_JACKPTH_LOCK, J2 +9V, J20 POWER_JACKPTH_LOCK, J21 POWER_JACKPTH_LOCK, J22 POWER_JACKPTH_LOCK, J23 POWER_JACKPTH_LOCK, J24 POWER_JACKPTH_LOCK, J3 GND, J4 POWER_JACKPTH_LOCK, J5 POWER_JACKPTH_LOCK, J6 POWER_JACKPTH_LOCK, J7 POWER_JACKPTH_LOCK, J8 POWER_JACKPTH_LOCK, J9 POWER_JACKPTH_LOCK, SW1 450301014042, SW2 450301014042, U1 ADS1299IPAG, U10 TPD4E1B06DCKR, U11 TPD4E1B06DCKR, U12 TPD4E1B06DCKR, U13 TPD4E1B06DCKR, U14 TPD4E1B06DCKR, U15 TPD4E1B06DCKR, U16 TPD4E1B06DCKR, U17 TPD4E1B06DCKR, U2 ADS1299IPAG, U3 LM62435BPPQRJRRQ1, U5 LP2982IM5-3.3/NOPB, U6 TPD4E1B06DCKR, U7 TPD4E1B06DCKR, U8 TPD4E1B06DCKR, U9 TPD4E1B06DCKR

Commit message: Add files via upload
Parts:
- moved R11 5.00 mm to (30.9, 18.9)
- moved R8 5.00 mm to (18.9, 19.0)
- moved R9 5.00 mm to (22.9, 18.9)
- moved R10 5.00 mm to (26.9, 18.9)
- moved R15 1.60 mm to (96.1, 8.92)
- moved D7 1.60 mm to (96.1, 4.67)
- moved D6 0.50 mm to (92.1, 4.67)
- moved R17 0.41 mm to (92.0, 8.92)
- moved R16 0.41 mm to (88.0, 8.92)
- moved D5 0.40 mm to (88.0, 4.67)
- moved D3 0.23 mm to (27.1, 13.8), turned to 270 degrees
- moved D4 0.21 mm to (31.0, 13.8), turned to 270 degrees
- moved D2 0.20 mm to (23.1, 13.9), turned to 270 degrees
- moved D1 0.18 mm to (19.1, 14.0), turned to 270 degrees
Routing:
- net GND: track 128.6 -> 133.0 mm
- net +3.3V-MBED: track 113.4 -> 115.4 mm
- net +9V: track 83.0 -> 81.4 mm
- net DEBUG_1: track 52.0 -> 53.7 mm
- net 9V_LED: track 4.34 -> 3.35 mm
- net 5V_LED: track 4.28 -> 3.38 mm
- net 3.3_ANA_LED: track 4.22 -> 3.42 mm
- net 3.3V_DIG_LED: track 4.16 -> 3.44 mm
Other:
- board text added: "+"
- board text added: "-"
- board text added: "3.3VM"
- board text added: "3.3VR"
- board text added: "BLE_EN"
- board text added: "DBG1"
- board text added: "DBG2"
- board text added: "DBG3"
- board text added: "Fall 2021"
- board text added: "GND"
- board text added: "Wireless Low Cost EEG Cap"
- board text removed: "3.3V-REG"
