File: EEG_cap_final.sch (EAGLE design)
At the start: 150 parts, among them J1 2908-05WB-MG, J10 POWER_JACKPTH_LOCK, J11 POWER_JACKPTH_LOCK, J12 POWER_JACKPTH_LOCK, J13 POWER_JACKPTH_LOCK, J14 POWER_JACKPTH_LOCK, J15 POWER_JACKPTH_LOCK, J16 POWER_JACKPTH_LOCK, J17 POWER_JACKPTH_LOCK, J18 POWER_JACKPTH_LOCK, J19 POWER_JACKPTH_LOCK, J2 +9V, J20 POWER_JACKPTH_LOCK, J21 POWER_JACKPTH_LOCK, J22 POWER_JACKPTH_LOCK, J23 POWER_JACKPTH_LOCK, J24 POWER_JACKPTH_LOCK, J3 GND, J4 POWER_JACKPTH_LOCK, J5 POWER_JACKPTH_LOCK, J6 POWER_JACKPTH_LOCK, J7 POWER_JACKPTH_LOCK, J8 POWER_JACKPTH_LOCK, J9 POWER_JACKPTH_LOCK, SW1 450301014042, SW2 450301014042, U1 ADS1299IPAG, U10 TPD4E1B06DCKR, U11 TPD4E1B06DCKR, U12 TPD4E1B06DCKR, U13 TPD4E1B06DCKR, U14 TPD4E1B06DCKR, U15 TPD4E1B06DCKR, U16 TPD4E1B06DCKR, U17 TPD4E1B06DCKR, U2 ADS1299IPAG, U3 LM62435BPPQRJRRQ1, U5 LP2982IM5-3.3/NOPB, U6 TPD4E1B06DCKR, U7 TPD4E1B06DCKR, U8 TPD4E1B06DCKR, U9 TPD4E1B06DCKR

Commit message: Add files via upload
Changed lines of the file:
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@@
 <attribute name="VALUE" x="390.8806" y="255.4986" size="2.0828" layer="96" ratio="6" rot="SR0"/>
 </instance>
-<instance part="SUPPLY49" gate="G$1" x="381" y="233.68" smashed="yes">
-<attribute name="VALUE" x="378.46" y="231.14" size="1.778" layer="96"/>
+<instance part="SUPPLY49" gate="G$1" x="381" y="231.14" smashed="yes">
+<attribute name="VALUE" x="378.46" y="228.6" size="1.778" layer="96"/>
 </instance>
 <instance part="RA5" gate="A" x="238.76" y="254" smashed="yes">
@@
 <attribute name="VALUE" x="390.8806" y="227.5586" size="2.0828" layer="96" ratio="6" rot="SR0"/>
 </instance>
-<instance part="SUPPLY62" gate="G$1" x="381" y="205.74" smashed="yes">
-<attribute name="VALUE" x="378.46" y="203.2" size="1.778" layer="96"/>
+<instance part="SUPPLY62" gate="G$1" x="381" y="203.2" smashed="yes">
+<attribute name="VALUE" x="378.46" y="200.66" size="1.778" layer="96"/>
 </instance>
 <instance part="J5" gate="G$1" x="391.16" y="182.88" smashed="yes">
@@
 <wire x1="381" y1="241.3" x2="383.54" y2="241.3" width="0.1524" layer="91"/>
 <pinref part="SUPPLY49" gate="G$1" pin="GND"/>
-<wire x1="381" y1="236.22" x2="381" y2="241.3" width="0.1524" layer="91"/>
+<wire x1="381" y1="233.68" x2="381" y2="241.3" width="0.1524" layer="91"/>
 <junction x="381" y="241.3"/>
 </segment>
@@
 <wire x1="381" y1="213.36" x2="383.54" y2="213.36" width="0.1524" layer="91"/>
 <pinref part="SUPPLY62" gate="G$1" pin="GND"/>
-<wire x1="381" y1="208.28" x2="381" y2="213.36" width="0.1524" layer="91"/>
+<wire x1="381" y1="205.74" x2="381" y2="213.36" width="0.1524" layer="91"/>
 <junction x="381" y="213.36"/>
 </segment>
@@
 </sheet>
 </sheets>
+<errors>
+</errors>
 </schematic>
 </drawing>
